Commit message: Start my own xacro journey

File: af_obstacle_avoidance_cpp/model/turtlebot3_waffle_pi.urdf (robot description, URDF)
Before this commit: robot turtlebot3_waffle, 13 links, 12 joints
Links:
- removed link base_laser_link
- removed link camera_depth_frame
- removed link camera_depth_optical_frame
- added link base_scan, mass 0.114; collision cylinder length=0.0315 radius=0.055; visual mesh filename=file://$(find af_obstacle_avoidance_cpp)/model/meshes/senso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 scale=0.001 0.001 0.001
- link camera_link: geometry collision box size=0.015 0.030 0.027
Joints:
- removed joint camera_depth_joint
- removed joint camera_depth_optical_joint
- removed joint laser_joint
- added joint scan_joint: type fixed, parent base_link, child base_scan, origin xyz=-0.064 0 0.122 rpy=0 0 0
- joint camera_joint: origin xyz=0.064 -0.065 0.094 rpy=0 0 0 -> xyz=0.073 -0.011 0.084 rpy=0 0 0
- joint camera_rgb_joint: origin xyz=${r200_cam_rgb_px} ${r200_cam_rgb_py} ${r200_cam_rgb_pz} rpy=0 0 0 -> xyz=0.003 0.011 0.009 rpy=0 0 0
