Commit message: Have to comment out the empty links or else parseURDF complain about too many root link. because a root link is empty so only base_footprint have to be empty

File: af_obstacle_avoidance_cpp/model/soheil.urdf.xacro (robot description, xacro)
@@ -3,13 +3,119 @@
     <link name="base_footprint"/>
     <link name="base_link">
+             <visual>
+                <origin xyz="-0.064 0 0.0" rpy="0 0 0"/>
+                <geometry>
+                    <mesh filename="file://$(find af_obstacle_avoidance_cpp)/model/meshes/bases/waffle_pi_base.stl" scale="0.001 0.001 0.001"/>
+                </geometry>
+                <material name="light_black"/>
+            </visual>
+            <collision>
+                <origin xyz="-0.064 0 0.047" rpy="0 0 0"/>
+                <geometry>
+                    <box size="0.266 0.266 0.094"/>
+                </geometry>
+            </collision>
+            <inertial>
+                <origin xyz="0 0 0" rpy="0 0 0"/>
+                <mass value="1.3729096e+00"/>
+                <inertia ixx="8.7002718e-03" ixy="-4.7576583e-05" ixz="1.1160499e-04"
+                        iyy="8.6195418e-03" iyz="-3.5422299e-06"
+                        izz="1.4612727e-02" />
+            </inertial>
     </link>
+<!--
     <link name="imu_link">
     </link>
     <link name="base_scan">
-    </link>
+    </link> -->
     <link name="wheel_left_link">
+        <visual>
+            <origin xyz="0 0 0" rpy="1.57 0 0"/>
+            <geometry>
+                <mesh filename="file://$(find af_obstacle_avoidance_cpp)/model/meshes/wheels/left_tire.stl" scale="0.001 0.001 0.001"/>
+            </geometry>
+            <material name="dark"/>
+        </visual>
+        <collision>
+            <origin xyz="0 0 0" rpy="0 0 0"/>
+            <geometry>
+                <cylinder length="0.018" radius="0.033"/>
+            </geometry>
+             <surface>
+            <!-- This friction pamareter don't contain reliable data!! -->
+            <friction>
+                <ode>
+                <mu>100000</mu>
+                <mu2>100000</mu2>
+                <fdir1>0 0 0</fdir1>
+                <slip1>0.0</slip1>
+                <slip2>0.0</slip2>
+                </ode>
+            </friction>
+            <contact>
+                <ode>
+                <soft_cfm>0</soft_cfm>
+                <soft_erp>0.2</soft_erp>
+                <kp>1e+5</kp>
+                <kd>1</kd>
+                <max_vel>0.01</max_vel>
+                <min_depth>0.001</min_depth>
+                </ode>
+            </contact>
+            </surface>
+        </collision>
+        <inertial>
+            <origin xyz="0 0 0" />
+            <mass value="2.8498940e-02" />
+            <inertia ixx="1.1175580e-05" ixy="-4.2369783e-11" ixz="-5.9381719e-09"
+                    iyy="1.1192413e-05" iyz="-1.4400107e-11"
+                    izz="2.0712558e-05" />
+        </inertial>
     </link>
     <link name="wheel_right_link">
+         <visual>
+            <origin xyz="0 0 0" rpy="1.57 0 0"/>
+            <geometry>
+                <mesh filename="file://$(find af_obstacle_avoidance_cpp)/model/meshes/wheels/right_tire.stl" scale="0.001 0.001 0.001"/>
+            </geometry>
+            <material name="dark"/>
+        </visual>
+        <collision>
+            <origin xyz="0 0 0" rpy="0 0 0"/>
+            <geometry>
+                <cylinder length="0.018" radius="0.033"/>
+            </geometry>
+            <surface>
+                <!-- This friction pamareter don't contain reliable data!! -->
+                <friction>
+                    <ode>
+                    <mu>100000</mu>
+                    <mu2>100000</mu2>
+                    <fdir1>0 0 0</fdir1>
+                    <slip1>0.0</slip1>
+                    <slip2>0.0</slip2>
+                    </ode>
+                </friction>
+                <contact>
+                    <ode>
+                    <soft_cfm>0</soft_cfm>
+                    <soft_erp>0.2</soft_erp>
+                    <kp>1e+5</kp>
+                    <kd>1</kd>
+                    <max_vel>0.01</max_vel>
+                    <min_depth>0.001</min_depth>
+                    </ode>
+                </contact>
+            </surface>
+        </collision>
+        <inertial>
+            <origin xyz="0 0 0" />
+            <mass value="2.8498940e-02" />
+            <inertia ixx="1.1175580e-05" ixy="-4.2369783e-11" ixz="-5.9381719e-09"
+                    iyy="1.1192413e-05" iyz="-1.4400107e-11"
+                    izz="2.0712558e-05" />
+        </inertial>
     </link>
+<!--
     <link name="caster_back_left_link">
     </link>
@@ -18,4 +124,24 @@
     <link name="camera_link"/>
     <link name="camera_rgb_optical_frame">
-    </link>
+    </link> -->
+    <!-- %%%%%%%%%%%%%%%%%%%%%%%%%%%%%% JOINTS%%%%%%%%%%%%%%%%%%%% -->
+    <joint name="base_joint" type="fixed">
+        <parent link="base_footprint"/>
+        <child link="base_link"/>
+        <origin xyz="0 0 0" rpy="0 0.01 0"/>
+    </joint>
+    <joint name="wheel_left_joint" type="revolute">
+        <parent link="base_link"/>
+        <child link="wheel_left_link"/>
+        <pose xyz="0 0 0.144" rpy="0.023 -1.57 0 0"/>
+        <axis xyz="0 0 1"/>
+        <limit effort="100" velocity="5" lower="-3.14" upper="3.14"/>
+    </joint>
+   <joint name="wheel_right_joint" type="revolute">
+        <parent link="base_link"/>
+        <child link="wheel_right_link"/>
+        <pose xyz="0 0 -0.144" rpy="0.023 -1.57 0 0"/>
+        <axis xyz="0 0 1"/>
+        <limit effort="100" velocity="5" lower="-3.14" upper="3.14"/>
+    </joint>
 </robot>

Commit message: Fix some bugs like using pose instead of origin in one of the wheels tag

File: af_obstacle_avoidance_cpp/model/soheil.urdf.xacro (robot description, xacro)
@@ -117,10 +117,59 @@
         </inertial>
     </link>
-<!--
     <link name="caster_back_left_link">
+        <collision>
+            <origin xyz="0 0.001 0" rpy="0 0 0"/>
+            <geometry>
+                <box size="0.030 0.009 0.020"/>
+            </geometry>
+            <surface>
+            <contact>
+                <ode>
+                <soft_cfm>0</soft_cfm>
+                <soft_erp>0.2</soft_erp>
+                <kp>1e+5</kp>
+                <kd>1</kd>
+                <max_vel>0.01</max_vel>
+                <min_depth>0.001</min_depth>
+                </ode>
+            </contact>
+            </surface>
+        </collision>
+        <inertial>
+        <origin xyz="0 0 0" />
+        <mass value="0.005" />
+        <inertia ixx="0.001" ixy="0.0" ixz="0.0"
+                iyy="0.001" iyz="0.0"
+                izz="0.001" />
+        </inertial>
     </link>
     <link name="caster_back_right_link">
-    </link>
-    <link name="camera_link"/>
+        <collision>
+            <origin xyz="0 0.001 0" rpy="0 0 0"/>
+            <geometry>
+                <box size="0.030 0.009 0.020"/>
+            </geometry>
+            <surface>
+            <contact>
+                <ode>
+                <soft_cfm>0</soft_cfm>
+                <soft_erp>0.2</soft_erp>
+                <kp>1e+5</kp>
+                <kd>1</kd>
+                <max_vel>0.01</max_vel>
+                <min_depth>0.001</min_depth>
+                </ode>
+            </contact>
+            </surface>
+        </collision>
+        <inertial>
+        <origin xyz="0 0 0" />
+        <mass value="0.005" />
+        <inertia ixx="0.001" ixy="0.0" ixz="0.0"
+                iyy="0.001" iyz="0.0"
+                izz="0.001" />
+        </inertial>
+    </link>
+    <!-- <link name="camera_link"/>
     <link name="camera_rgb_optical_frame">
     </link> -->
@@ -134,5 +183,5 @@
         <parent link="base_link"/>
         <child link="wheel_left_link"/>
-        <pose xyz="0 0 0.144" rpy="0.023 -1.57 0 0"/>
+        <origin xyz="0.0 0.144 0.023" rpy="-1.57 0 0"/>
         <axis xyz="0 0 1"/>
         <limit effort="100" velocity="5" lower="-3.14" upper="3.14"/>
@@ -141,7 +190,15 @@
         <parent link="base_link"/>
         <child link="wheel_right_link"/>
-        <pose xyz="0 0 -0.144" rpy="0.023 -1.57 0 0"/>
+        <origin xyz="0.0 -0.144 0.023" rpy="-1.57 0 0"/>
         <axis xyz="0 0 1"/>
         <limit effort="100" velocity="5" lower="-3.14" upper="3.14"/>
     </joint>
+   <joint name='caster_back_right_joint' type='fixed'>
+        <parent link="base_link"/>
+        <child link="caster_back_right_link"/>
+    </joint>
+   <joint name='caster_back_left_joint' type='fixed'>
+        <parent link="base_link"/>
+        <child link="caster_back_left_link"/>
+    </joint>
 </robot>

Commit message: Add imu link and joint and the data is published thorugh tf_static. this is also true for caster_left and right

File: af_obstacle_avoidance_cpp/model/soheil.urdf.xacro (robot description, xacro)
@@ -24,8 +24,59 @@
             </inertial>
     </link>
-<!--
     <link name="imu_link">
-    </link>
-    <link name="base_scan">
+        <sensor name="tb3_imu" type="imu">
+            <always_on>true</always_on>
+            <update_rate>200</update_rate>
+            <imu>
+            <angular_velocity>
+                <x>
+                <noise type="gaussian">
+                    <mean>0.0</mean>
+                    <stddev>2e-4</stddev>
+                </noise>
+                </x>
+                <y>
+                <noise type="gaussian">
+                    <mean>0.0</mean>
+                    <stddev>2e-4</stddev>
+                </noise>
+                </y>
+                <z>
+                <noise type="gaussian">
+                    <mean>0.0</mean>
+                    <stddev>2e-4</stddev>
+                </noise>
+                </z>
+            </angular_velocity>
+            <linear_acceleration>
+                <x>
+                <noise type="gaussian">
+                    <mean>0.0</mean>
+                    <stddev>1.7e-2</stddev>
+                </noise>
+                </x>
+                <y>
+                <noise type="gaussian">
+                    <mean>0.0</mean>
+                    <stddev>1.7e-2</stddev>
+                </noise>
+                </y>
+                <z>
+                <noise type="gaussian">
+                    <mean>0.0</mean>
+                    <stddev>1.7e-2</stddev>
+                </noise>
+                </z>
+            </linear_acceleration>
+            </imu>
+            <plugin name="turtlebot3_imu" filename="libgazebo_ros_imu_sensor.so">
+            <ros>
+                <!-- <namespace>/tb3</namespace> -->
+                <remapping>~/out:=imu</remapping>
+            </ros>
+            </plugin>
+      </sensor>
+    </link>
+    <!-- <link name="base_scan">
     </link> -->
     <link name="wheel_left_link">
@@ -202,3 +253,9 @@
         <child link="caster_back_left_link"/>
     </joint>
+    <joint name="imu_joint" type="fixed">
+        <parent link="base_link"/>
+        <child link="imu_link"/>
+        <origin xyz="-0.032 0 0.068 " rpy="0 0 0"/>
+        <axis xyz="0 0 1"/>
+    </joint>
 </robot>

Commit message: Just to simulate the too many roots error, the problem is defining a joint for all the links except the root link!

File: af_obstacle_avoidance_cpp/model/soheil.urdf.xacro (robot description, xacro)
@@ -78,6 +78,60 @@
       </sensor>
     </link>
-    <!-- <link name="base_scan">
-    </link> -->
+    <link name="base_scan">
+        <visual>
+            <origin xyz="0 0 0" rpy="0 0 0"/>
+            <geometry>
+                <mesh filename="file://$(find af_obstacle_avoidance_cpp)/model/meshes/sensors/lds.stl" scale="0.001 0.001 0.001"/>
+            </geometry>
+            <material name="dark"/>
+        </visual>
+        <collision>
+        <origin xyz="0.015 0 -0.0065" rpy="0 0 0"/>
+        <geometry>
+            <cylinder length="0.0315" radius="0.055"/>
+        </geometry>
+        </collision>
+        <inertial>
+        <mass value="0.114" />
+        <origin xyz="0 0 0" />
+        <inertia ixx="0.001" ixy="0.0" ixz="0.0"
+                iyy="0.001" iyz="0.0"
+                izz="0.001" />
+        </inertial>
+        <sensor name="hls_lfcd_lds" type="ray">
+            <always_on>true</always_on>
+            <visualize>true</visualize>
+            <pose>-0.064 0 0.121 0 0 0</pose>
+            <update_rate>5</update_rate>
+            <ray>
+            <scan>
+                <horizontal>
+                <samples>360</samples>
+                <resolution>1.000000</resolution>
+                <min_angle>0.000000</min_angle>
+                <max_angle>6.280000</max_angle>
+                </horizontal>
+            </scan>
+            <range>
+                <min>0.120000</min>
+                <max>3.5</max>
+                <resolution>0.015000</resolution>
+            </range>
+            <noise>
+                <type>gaussian</type>
+                <mean>0.0</mean>
+                <stddev>0.01</stddev>
+            </noise>
+            </ray>
+            <plugin name="turtlebot3_laserscan" filename="libgazebo_ros_ray_sensor.so">
+            <ros>
+                <!-- <namespace>/tb3</namespace> -->
+                <remapping>~/out:=scan</remapping>
+            </ros>
+            <output_type>sensor_msgs/LaserScan</output_type>
+            <frame_name>base_scan</frame_name>
+            </plugin>
+        </sensor>
+    </link>
     <link name="wheel_left_link">
         <visual>
@@ -259,3 +313,9 @@
         <axis xyz="0 0 1"/>
     </joint>
+    <!-- <joint name="lidar_joint" type="fixed">
+        <parent link="base_link"/>
+        <child link="base_scan"/>
+        <origin xyz="-0.064 0 0.121" rpy="0 0 0"/>
+        <axis xyz="0 0 1"/>
+    </joint> -->
 </robot>

Commit message: Add a lidar and now the robot slips on the floor

File: af_obstacle_avoidance_cpp/model/soheil.urdf.xacro (robot description, xacro)
@@ -87,5 +87,5 @@
         </visual>
         <collision>
-        <origin xyz="0.015 0 -0.0065" rpy="0 0 0"/>
+        <origin xyz="0.0 0 0.0" rpy="0 0 0"/>
         <geometry>
             <cylinder length="0.0315" radius="0.055"/>
@@ -313,9 +313,9 @@
         <axis xyz="0 0 1"/>
     </joint>
-    <!-- <joint name="lidar_joint" type="fixed">
+    <joint name="lidar_joint" type="fixed">
         <parent link="base_link"/>
         <child link="base_scan"/>
         <origin xyz="-0.064 0 0.121" rpy="0 0 0"/>
         <axis xyz="0 0 1"/>
-    </joint> -->
+    </joint>
 </robot>
