Commit message: Wrong xacro, in gazebo turn on contact in view in the menu bar to see and compare it to the original tb3 and you'll see whats wrong!

File: af_obstacle_avoidance_cpp/model/soheil.urdf.xacro (robot description, xacro)
@@ -1,4 +1,14 @@
 <?xml version="1.0"?>
-<robot name = "turtlebot3_waffle_pi" xmlns:xacro="http://ros.org/wiki/xacro">
+<robot name = "turtlebot4_waffle_pi" xmlns:xacro="http://ros.org/wiki/xacro">
+  <!-- Init colour -->
+  <material name="black">
+      <color rgba="0.0 0.0 0.0 1.0"/>
+  </material>
+  <material name="dark">
+    <color rgba="0.3 0.3 0.3 1.0"/>
+  </material>
+  <material name="light_black">
+    <color rgba="0.4 0.4 0.4 1.0"/>
+  </material>
     <link name="base_footprint"/>
     <link name="base_link">
@@ -25,56 +35,4 @@
     </link>
     <link name="imu_link">
-        <sensor name="tb3_imu" type="imu">
-            <always_on>true</always_on>
-            <update_rate>200</update_rate>
-            <imu>
-            <angular_velocity>
-                <x>
-                <noise type="gaussian">
-                    <mean>0.0</mean>
-                    <stddev>2e-4</stddev>
-                </noise>
-                </x>
-                <y>
-                <noise type="gaussian">
-                    <mean>0.0</mean>
-                    <stddev>2e-4</stddev>
-                </noise>
-                </y>
-                <z>
-                <noise type="gaussian">
-                    <mean>0.0</mean>
-                    <stddev>2e-4</stddev>
-                </noise>
-                </z>
-            </angular_velocity>
-            <linear_acceleration>
-                <x>
-                <noise type="gaussian">
-                    <mean>0.0</mean>
-                    <stddev>1.7e-2</stddev>
-                </noise>
-                </x>
-                <y>
-                <noise type="gaussian">
-                    <mean>0.0</mean>
-                    <stddev>1.7e-2</stddev>
-                </noise>
-                </y>
-                <z>
-                <noise type="gaussian">
-                    <mean>0.0</mean>
-                    <stddev>1.7e-2</stddev>
-                </noise>
-                </z>
-            </linear_acceleration>
-            </imu>
-            <plugin name="turtlebot3_imu" filename="libgazebo_ros_imu_sensor.so">
-            <ros>
-                <!-- <namespace>/tb3</namespace> -->
-                <remapping>~/out:=imu</remapping>
-            </ros>
-            </plugin>
-      </sensor>
     </link>
     <link name="base_scan">
@@ -99,5 +57,205 @@
                 izz="0.001" />
         </inertial>
-        <sensor name="hls_lfcd_lds" type="ray">
+    </link>
+    <link name="wheel_left_link">
+        <visual>
+            <origin xyz="0 0 0" rpy="1.57 0 0"/>
+            <geometry>
+                <mesh filename="file://$(find af_obstacle_avoidance_cpp)/model/meshes/wheels/left_tire.stl" scale="0.001 0.001 0.001"/>
+            </geometry>
+            <material name="dark"/>
+        </visual>
+        <collision>
+            <origin xyz="0 0 0" rpy="0 0 0"/>
+            <geometry>
+                <cylinder length="0.018" radius="0.033"/>
+            </geometry>
+        </collision>
+        <inertial>
+            <origin xyz="0 0 0" />
+            <mass value="2.8498940e-02" />
+            <inertia ixx="1.1175580e-05" ixy="-4.2369783e-11" ixz="-5.9381719e-09"
+                    iyy="1.1192413e-05" iyz="-1.4400107e-11"
+                    izz="2.0712558e-05" />
+        </inertial>
+    </link>
+    <link name="wheel_right_link">
+         <visual>
+            <origin xyz="0 0 0" rpy="1.57 0 0"/>
+            <geometry>
+                <mesh filename="file://$(find af_obstacle_avoidance_cpp)/model/meshes/wheels/right_tire.stl" scale="0.001 0.001 0.001"/>
+            </geometry>
+            <material name="dark"/>
+        </visual>
+        <collision>
+            <origin xyz="0 0 0" rpy="0 0 0"/>
+            <geometry>
+                <cylinder length="0.018" radius="0.033"/>
+            </geometry>
+        </collision>
+        <inertial>
+            <origin xyz="0 0 0" />
+            <mass value="2.8498940e-02" />
+            <inertia ixx="1.1175580e-05" ixy="-4.2369783e-11" ixz="-5.9381719e-09"
+                    iyy="1.1192413e-05" iyz="-1.4400107e-11"
+                    izz="2.0712558e-05" />
+        </inertial>
+    </link>
+    <link name="caster_back_left_link">
+        <collision>
+            <origin xyz="0 0.001 0" rpy="0 0 0"/>
+            <geometry>
+                <box size="0.030 0.009 0.020"/>
+            </geometry>
+        </collision>
+        <inertial>
+        <origin xyz="0 0 0" />
+        <mass value="0.005" />
+        <inertia ixx="0.001" ixy="0.0" ixz="0.0"
+                iyy="0.001" iyz="0.0"
+                izz="0.001" />
+        </inertial>
+    </link>
+    <link name="caster_back_right_link">
+        <collision>
+            <origin xyz="0 0.001 0" rpy="0 0 0"/>
+            <geometry>
+                <box size="0.030 0.009 0.020"/>
+            </geometry>
+        </collision>
+        <inertial>
+        <origin xyz="0 0 0" />
+        <mass value="0.005" />
+        <inertia ixx="0.001" ixy="0.0" ixz="0.0"
+                iyy="0.001" iyz="0.0"
+                izz="0.001" />
+        </inertial>
+    </link>
+    <!-- <link name="camera_link"/>
+    <link name="camera_rgb_optical_frame">
+    </link> -->
+    <!-- %%%%%%%%%%%%%%%%%%%%%%%%%%%%%% JOINTS%%%%%%%%%%%%%%%%%%%% -->
+    <joint name="base_joint" type="fixed">
+        <parent link="base_footprint"/>
+        <child link="base_link"/>
+        <origin xyz="0 0 0" rpy="0 0.01 0"/>
+    </joint>
+    <joint name="wheel_left_joint" type="revolute">
+        <parent link="base_link"/>
+        <child link="wheel_left_link"/>
+        <origin xyz="0.0 0.144 0.023" rpy="-1.57 0 0"/>
+        <axis xyz="0 0 1"/>
+        <limit effort="100" velocity="5" lower="-3.14" upper="3.14"/>
+    </joint>
+   <joint name="wheel_right_joint" type="revolute">
+        <parent link="base_link"/>
+        <child link="wheel_right_link"/>
+        <origin xyz="0.0 -0.144 0.023" rpy="-1.57 0 0"/>
+        <axis xyz="0 0 1"/>
+        <limit effort="100" velocity="5" lower="-3.14" upper="3.14"/>
+    </joint>
+   <joint name='caster_back_right_joint' type='fixed'>
+        <parent link="base_link"/>
+        <child link="caster_back_right_link"/>
+    </joint>
+   <joint name='caster_back_left_joint' type='fixed'>
+        <parent link="base_link"/>
+        <child link="caster_back_left_link"/>
+    </joint>
+    <joint name="imu_joint" type="fixed">
+        <parent link="base_link"/>
+        <child link="imu_link"/>
+        <origin xyz="-0.032 0 0.068 " rpy="0 0 0"/>
+        <axis xyz="0 0 1"/>
+    </joint>
+    <joint name="lidar_joint" type="fixed">
+        <parent link="base_link"/>
+        <child link="base_scan"/>
+        <origin xyz="-0.064 0 0.121" rpy="0 0 0"/>
+        <axis xyz="0 0 1"/>
+    </joint>
+    <!-- Publish odom and base_footprint in tf topic  -->
+    <gazebo>
+        <plugin name="turtlebot3_diff_drive" filename="libgazebo_ros_diff_drive.so">
+            <ros>
+                <!-- <namespace>/tb3</namespace> -->
+            </ros>
+            <update_rate>30</update_rate>
+            <!-- wheels -->
+            <left_joint>wheel_left_joint</left_joint>
+            <right_joint>wheel_right_joint</right_joint>
+            <!-- kinematics -->
+            <wheel_separation>0.287</wheel_separation>
+            <wheel_diameter>0.066</wheel_diameter>
+            <!-- limits -->
+            <max_wheel_torque>200</max_wheel_torque>
+            <max_wheel_acceleration>1.0</max_wheel_acceleration>
+            <command_topic>cmd_vel</command_topic>
+            <!-- output -->
+            <publish_odom>true</publish_odom>
+            <publish_odom_tf>true</publish_odom_tf>
+            <publish_wheel_tf>false</publish_wheel_tf>
+            <odometry_topic>odom</odometry_topic>
+            <odometry_frame>odom</odometry_frame>
+            <robot_base_frame>base_footprint</robot_base_frame>
+        </plugin>
+    </gazebo>
+    <!-- To publish other frames besides odom and base_footprint to publish their tf transforms in the tf topic  -->
+    <gazebo>
+        <plugin name="turtlebot3_joint_state" filename="libgazebo_ros_joint_state_publisher.so">
+            <ros>
+            <!-- <namespace>/tb3</namespace> -->
+                <remapping>~/out:=joint_states</remapping>
+            </ros>
+            <update_rate>30</update_rate>
+            <joint_name>wheel_left_joint</joint_name>
+            <joint_name>wheel_right_joint</joint_name>
+        </plugin>
+    </gazebo>
+  <gazebo reference="base_link">
+    <material>Gazebo/DarkGrey</material>
+  </gazebo>
+  <gazebo reference="wheel_left_link">
+    <mu1>100000</mu1>
+    <mu2>100000</mu2>
+    <kp>100000.0</kp>
+    <kd>1.0</kd>
+    <minDepth>0.001</minDepth>
+    <maxVel>0.1</maxVel>
+    <fdir1>0 0 0</fdir1>
+    <material>Gazebo/FlatBlack</material>
+  </gazebo>
+  <gazebo reference="wheel_right_link">
+    <mu1>100000</mu1>
+    <mu2>100000</mu2>
+    <kp>100000.0</kp>
+    <kd>1.0</kd>
+    <minDepth>0.001</minDepth>
+    <maxVel>0.1</maxVel>
+    <fdir1>0 0 0</fdir1>
+    <material>Gazebo/FlatBlack</material>
+  </gazebo>
+  <gazebo reference="caster_back_right_link">
+    <mu1>1.0</mu1>
+    <mu2>1.0</mu2>
+    <kp>100000.0</kp>
+    <kd>1.0</kd>
+    <minDepth>0.001</minDepth>
+    <maxVel>0.01</maxVel>
+    <material>Gazebo/White</material>
+  </gazebo>
+  <gazebo reference="caster_back_left_link">
+    <mu1>1.0</mu1>
+    <mu2>1.0</mu2>
+    <kp>100000.0</kp>
+    <kd>1.0</kd>
+    <minDepth>0.001</minDepth>
+    <maxVel>0.01</maxVel>
+    <material>Gazebo/White</material>
+  </gazebo>
+    <!-- in the scan topic -->
+    <gazebo reference="base_scan">
+        <material value="Gazebo/FlatBlack"/>
+       <sensor name="hls_lfcd_lds" type="ray">
             <always_on>true</always_on>
             <visualize>true</visualize>
@@ -126,5 +284,4 @@
             <plugin name="turtlebot3_laserscan" filename="libgazebo_ros_ray_sensor.so">
             <ros>
-                <!-- <namespace>/tb3</namespace> -->
                 <remapping>~/out:=scan</remapping>
             </ros>
@@ -133,189 +290,59 @@
             </plugin>
         </sensor>
-    </link>
-    <link name="wheel_left_link">
-        <visual>
-            <origin xyz="0 0 0" rpy="1.57 0 0"/>
-            <geometry>
-                <mesh filename="file://$(find af_obstacle_avoidance_cpp)/model/meshes/wheels/left_tire.stl" scale="0.001 0.001 0.001"/>
-            </geometry>
-            <material name="dark"/>
-        </visual>
-        <collision>
-            <origin xyz="0 0 0" rpy="0 0 0"/>
-            <geometry>
-                <cylinder length="0.018" radius="0.033"/>
-            </geometry>
-             <surface>
-            <!-- This friction pamareter don't contain reliable data!! -->
-            <friction>
-                <ode>
-                <mu>100000</mu>
-                <mu2>100000</mu2>
-                <fdir1>0 0 0</fdir1>
-                <slip1>0.0</slip1>
-                <slip2>0.0</slip2>
-                </ode>
-            </friction>
-            <contact>
-                <ode>
-                <soft_cfm>0</soft_cfm>
-                <soft_erp>0.2</soft_erp>
-                <kp>1e+5</kp>
-                <kd>1</kd>
-                <max_vel>0.01</max_vel>
-                <min_depth>0.001</min_depth>
-                </ode>
-            </contact>
-            </surface>
-        </collision>
-        <inertial>
-            <origin xyz="0 0 0" />
-            <mass value="2.8498940e-02" />
-            <inertia ixx="1.1175580e-05" ixy="-4.2369783e-11" ixz="-5.9381719e-09"
-                    iyy="1.1192413e-05" iyz="-1.4400107e-11"
-                    izz="2.0712558e-05" />
-        </inertial>
-    </link>
-    <link name="wheel_right_link">
-         <visual>
-            <origin xyz="0 0 0" rpy="1.57 0 0"/>
-            <geometry>
-                <mesh filename="file://$(find af_obstacle_avoidance_cpp)/model/meshes/wheels/right_tire.stl" scale="0.001 0.001 0.001"/>
-            </geometry>
-            <material name="dark"/>
-        </visual>
-        <collision>
-            <origin xyz="0 0 0" rpy="0 0 0"/>
-            <geometry>
-                <cylinder length="0.018" radius="0.033"/>
-            </geometry>
-            <surface>
-                <!-- This friction pamareter don't contain reliable data!! -->
-                <friction>
-                    <ode>
-                    <mu>100000</mu>
-                    <mu2>100000</mu2>
-                    <fdir1>0 0 0</fdir1>
-                    <slip1>0.0</slip1>
-                    <slip2>0.0</slip2>
-                    </ode>
-                </friction>
-                <contact>
-                    <ode>
-                    <soft_cfm>0</soft_cfm>
-                    <soft_erp>0.2</soft_erp>
-                    <kp>1e+5</kp>
-                    <kd>1</kd>
-                    <max_vel>0.01</max_vel>
-                    <min_depth>0.001</min_depth>
-                    </ode>
-                </contact>
-            </surface>
-        </collision>
-        <inertial>
-            <origin xyz="0 0 0" />
-            <mass value="2.8498940e-02" />
-            <inertia ixx="1.1175580e-05" ixy="-4.2369783e-11" ixz="-5.9381719e-09"
-                    iyy="1.1192413e-05" iyz="-1.4400107e-11"
-                    izz="2.0712558e-05" />
-        </inertial>
-    </link>
-    <link name="caster_back_left_link">
-        <collision>
-            <origin xyz="0 0.001 0" rpy="0 0 0"/>
-            <geometry>
-                <box size="0.030 0.009 0.020"/>
-            </geometry>
-            <surface>
-            <contact>
-                <ode>
-                <soft_cfm>0</soft_cfm>
-                <soft_erp>0.2</soft_erp>
-                <kp>1e+5</kp>
-                <kd>1</kd>
-                <max_vel>0.01</max_vel>
-                <min_depth>0.001</min_depth>
-                </ode>
-            </contact>
-            </surface>
-        </collision>
-        <inertial>
-        <origin xyz="0 0 0" />
-        <mass value="0.005" />
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
Commit message: Type of the wheel joint  must be continuous not revolute!

File: af_obstacle_avoidance_cpp/model/soheil.urdf.xacro (robot description, xacro)
@@ -141,25 +141,25 @@
         <origin xyz="0 0 0" rpy="0 0.01 0"/>
     </joint>
-    <joint name="wheel_left_joint" type="revolute">
+    <joint name="wheel_left_joint" type="continuous">
         <parent link="base_link"/>
         <child link="wheel_left_link"/>
         <origin xyz="0.0 0.144 0.023" rpy="-1.57 0 0"/>
         <axis xyz="0 0 1"/>
-        <limit effort="100" velocity="5" lower="-3.14" upper="3.14"/>
-    </joint>
-   <joint name="wheel_right_joint" type="revolute">
+    </joint>
+   <joint name="wheel_right_joint" type="continuous">
         <parent link="base_link"/>
         <child link="wheel_right_link"/>
         <origin xyz="0.0 -0.144 0.023" rpy="-1.57 0 0"/>
         <axis xyz="0 0 1"/>
-        <limit effort="100" velocity="5" lower="-3.14" upper="3.14"/>
     </joint>
    <joint name='caster_back_right_joint' type='fixed'>
         <parent link="base_link"/>
         <child link="caster_back_right_link"/>
+        <origin xyz="-0.177 -0.064 -0.004" rpy="-1.57 0 0"/>
     </joint>
    <joint name='caster_back_left_joint' type='fixed'>
         <parent link="base_link"/>
         <child link="caster_back_left_link"/>
+        <origin xyz="-0.177 0.064 -0.004" rpy="-1.57 0 0"/>
     </joint>
     <joint name="imu_joint" type="fixed">
@@ -189,5 +189,5 @@
             <wheel_diameter>0.066</wheel_diameter>
             <!-- limits -->
-            <max_wheel_torque>200</max_wheel_torque>
+            <max_wheel_torque>10</max_wheel_torque>
             <max_wheel_acceleration>1.0</max_wheel_acceleration>
             <command_topic>cmd_vel</command_topic>
@@ -217,40 +217,40 @@
   </gazebo>
   <gazebo reference="wheel_left_link">
-    <mu1>100000</mu1>
-    <mu2>100000</mu2>
-    <kp>100000.0</kp>
-    <kd>1.0</kd>
+    <mu1>0.1</mu1>
+    <mu2>0.1</mu2>
+    <kp>500000.0</kp>
+    <kd>10.0</kd>
     <minDepth>0.001</minDepth>
     <maxVel>0.1</maxVel>
-    <fdir1>0 0 0</fdir1>
+    <fdir1>1 0 0</fdir1>
     <material>Gazebo/FlatBlack</material>
   </gazebo>
   <gazebo reference="wheel_right_link">
-    <mu1>100000</mu1>
-    <mu2>100000</mu2>
-    <kp>100000.0</kp>
-    <kd>1.0</kd>
+    <mu1>0.1</mu1>
+    <mu2>0.1</mu2>
+    <kp>500000.0</kp>
+    <kd>10.0</kd>
     <minDepth>0.001</minDepth>
     <maxVel>0.1</maxVel>
-    <fdir1>0 0 0</fdir1>
+    <fdir1>1 0 0</fdir1>
     <material>Gazebo/FlatBlack</material>
   </gazebo>
   <gazebo reference="caster_back_right_link">
-    <mu1>1.0</mu1>
-    <mu2>1.0</mu2>
-    <kp>100000.0</kp>
-    <kd>1.0</kd>
+    <mu1>0.1</mu1>
+    <mu2>0.1</mu2>
+    <kp>1000000.0</kp>
+    <kd>100.0</kd>
     <minDepth>0.001</minDepth>
-    <maxVel>0.01</maxVel>
-    <material>Gazebo/White</material>
+    <maxVel>1.0</maxVel>
+    <material>Gazebo/FlatBlack</material>
   </gazebo>
   <gazebo reference="caster_back_left_link">
-    <mu1>1.0</mu1>
-    <mu2>1.0</mu2>
-    <kp>100000.0</kp>
-    <kd>1.0</kd>
+    <mu1>0.1</mu1>
+    <mu2>0.1</mu2>
+    <kp>1000000.0</kp>
+    <kd>100.0</kd>
     <minDepth>0.001</minDepth>
-    <maxVel>0.01</maxVel>
-    <material>Gazebo/White</material>
+    <maxVel>1.0</maxVel>
+    <material>Gazebo/FlatBlack</material>
   </gazebo>
     <!-- in the scan topic -->

File: af_obstacle_avoidance_cpp/model/soso.urdf (robot description, URDF)
Before this commit: robot turtlebot3_waffle, 13 links, 12 joints
Links:
- removed link base_laser_link
- removed link camera_depth_frame
- removed link camera_depth_optical_frame
- removed link camera_link
- removed link camera_rgb_frame
- removed link camera_rgb_optical_frame
- added link base_scan, mass 0.114; collision cylinder length=0.0315 radius=0.055; visual mesh filename=file:///home/course/Ros2Basics/install/af_obstacle_avoidanc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 scale=0.001 0.001 0.001
Joints:
- removed joint camera_depth_joint
- removed joint camera_depth_optical_joint
- removed joint camera_joint
- removed joint camera_rgb_joint
- removed joint camera_rgb_optical_joint
- removed joint laser_joint
- added joint lidar_joint: type fixed, parent base_link, child base_scan, origin xyz=-0.064 0 0.121 rpy=0 0 0, axis 0 0 1
- joint base_joint: origin xyz=0 0 0.010 rpy=0 0 0 -> xyz=0 0 0 rpy=0 0.01 0
- joint imu_joint: axis (none) -> 0 0 1; origin xyz=0.0 0 0.068 rpy=0 0 0 -> xyz=-0.032 0 0.068  rpy=0 0 0
- joint wheel_left_joint: limit (none) -> lower=-3.14 upper=3.14 effort=100 velocity=5; type continuous -> revolute
- joint wheel_right_joint: limit (none) -> lower=-3.14 upper=3.14 effort=100 velocity=5; type continuous -> revolute
