Commit message: Add camera

File: af_obstacle_avoidance_cpp/model/soheil.urdf.xacro (robot description, xacro)
@@ -132,7 +132,7 @@
         </inertial>
     </link>
-    <!-- <link name="camera_link"/>
-    <link name="camera_rgb_optical_frame">
-    </link> -->
+    <link name="camera_link"/>
+    <link name="camera_rgb_frame"/>
+    <link name="camera_rgb_optical_frame"/>
     <!-- %%%%%%%%%%%%%%%%%%%%%%%%%%%%%% JOINTS%%%%%%%%%%%%%%%%%%%% -->
     <joint name="base_joint" type="fixed">
@@ -141,4 +141,9 @@
         <origin xyz="0 0 0" rpy="0 0.01 0"/>
     </joint>
+    <!--
+        in xacro file its continuous but in sdf file its revolute (you can check model.sdf) and if you specify
+        revolute here it's wrong because then you have to specify limit and then the wheel
+        is gonna be restricted to the lower and higher angle and it won't roll continuously
+     -->
     <joint name="wheel_left_joint" type="continuous">
         <parent link="base_link"/>
@@ -175,4 +180,20 @@
         <axis xyz="0 0 1"/>
     </joint>
+    <joint name="camera_joint" type="fixed">
+        <parent link="base_link"/>
+        <child link="camera_link"/>
+        <origin xyz="0.073 -0.011 0.084" rpy="0 0 0"/>
+    </joint>
+    <joint name="camera_rgb_joint" type="fixed">
+        <parent link="camera_link"/>
+        <child link="camera_rgb_frame"/>
+        <origin xyz="0.003 0.011 0.009" rpy="0 0 0"/>
+    </joint>
+  <joint name="camera_rgb_optical_joint" type="fixed">
+    <origin xyz="0 0 0" rpy="-1.57 0 0"/>
+    <parent link="camera_rgb_frame"/>
+    <child link="camera_rgb_optical_frame"/>
+  </joint>
+<!-- %%%%%%%%%%%%%%%%%%%%%%%%%%%% gazebo tag %%%%%%%%%%%%%%%%%%%%%%%%%%%% -->
     <!-- Publish odom and base_footprint in tf topic  -->
     <gazebo>
@@ -202,4 +223,5 @@
     </gazebo>
     <!-- To publish other frames besides odom and base_footprint to publish their tf transforms in the tf topic  -->
+    <!-- I guess this is new in ros 2 and in ros 1 we didn't have to specify this explicitly  -->
     <gazebo>
         <plugin name="turtlebot3_joint_state" filename="libgazebo_ros_joint_state_publisher.so">
@@ -346,3 +368,53 @@
             </sensor>
     </gazebo>
+    <gazebo reference="camera_rgb_optical_frame">
+      <inertial>
+        <pose>0.076 0.0 0.093 0 0 0</pose>
+        <inertia>
+          <ixx>0.001</ixx>
+          <ixy>0.000</ixy>
+          <ixz>0.000</ixz>
+          <iyy>0.001</iyy>
+          <iyz>0.000</iyz>
+          <izz>0.001</izz>
+        </inertia>
+        <mass>0.035</mass>
+      </inertial>
+      <pose>0.076 0.0 0.093 0 0 0</pose>
+        <sensor name="camera" type="camera">
+                <always_on>true</always_on>
+                <visualize>true</visualize>
+                <update_rate>30</update_rate>
+                <camera name="picam">
+                <horizontal_fov>1.085595</horizontal_fov>
+                <image>
+                    <width>640</width>
+                    <height>480</height>
+                    <format>R8G8B8</format>
+                </image>
+                <clip>
+                    <near>0.03</near>
+                    <far>100</far>
+                </clip>
+                <noise>
+                    <type>gaussian</type>
+                    <!-- Noise is sampled independently per pixel on each frame.
+                        That pixel's noise value is added to each of its color
+                        channels, which at that point lie in the range [0,1]. -->
+                    <mean>0.0</mean>
+                    <stddev>0.007</stddev>
+                </noise>
+                </camera>
+                <plugin name="camera_driver" filename="libgazebo_ros_camera.so">
+                    <ros>
+                    <!-- <namespace>test_cam</namespace> -->
+                    <!-- <remapping>image_raw:=image_demo</remapping> -->
+                    <!-- <remapping>camera_info:=camera_info_demo</remapping> -->
+                    </ros>
+                    <!-- camera_name>omit so it defaults to sensor name</camera_name-->
+                    <!-- frame_name>omit so it defaults to link name</frameName-->
+                    <!-- <hack_baseline>0.07</hack_baseline> -->
+                </plugin>
+            </sensor>
+    </gazebo>
 </robot>
