Commit message: Add functionality

File: af_obstacle_avoidance_cpp/model/my_tb3.urdf.xacro (robot description, xacro)
@@ -1,4 +1,4 @@
 <?xml version="1.0"?>
-<robot name = "turtlebot4_waffle_pi" xmlns:xacro="http://ros.org/wiki/xacro">
+<robot name = "turtlebot3_waffle_pi" xmlns:xacro="http://ros.org/wiki/xacro">
   <!-- Init colour -->
   <material name="black">

File: af_obstacle_avoidance_py/model/my_tb3.urdf.xacro (robot description, xacro)
@@ -1,4 +1,4 @@
 <?xml version="1.0"?>
-<robot name = "turtlebot4_waffle_pi" xmlns:xacro="http://ros.org/wiki/xacro">
+<robot name = "turtlebot3_waffle_pi" xmlns:xacro="http://ros.org/wiki/xacro">
   <!-- Init colour -->
   <material name="black">
@@ -16,5 +16,5 @@
                 <origin xyz="-0.064 0 0.0" rpy="0 0 0"/>
                 <geometry>
-                    <mesh filename="file://$(find af_obstacle_avoidance_cpp)/model/meshes/bases/waffle_pi_base.stl" scale="0.001 0.001 0.001"/>
+                    <mesh filename="file://$(find af_obstacle_avoidance_py)/model/meshes/bases/waffle_pi_base.stl" scale="0.001 0.001 0.001"/>
                 </geometry>
                 <material name="light_black"/>
@@ -40,5 +40,5 @@
             <origin xyz="0 0 0" rpy="0 0 0"/>
             <geometry>
-                <mesh filename="file://$(find af_obstacle_avoidance_cpp)/model/meshes/sensors/lds.stl" scale="0.001 0.001 0.001"/>
+                <mesh filename="file://$(find af_obstacle_avoidance_py)/model/meshes/sensors/lds.stl" scale="0.001 0.001 0.001"/>
             </geometry>
             <material name="dark"/>
@@ -62,5 +62,5 @@
             <origin xyz="0 0 0" rpy="1.57 0 0"/>
             <geometry>
-                <mesh filename="file://$(find af_obstacle_avoidance_cpp)/model/meshes/wheels/left_tire.stl" scale="0.001 0.001 0.001"/>
+                <mesh filename="file://$(find af_obstacle_avoidance_py)/model/meshes/wheels/left_tire.stl" scale="0.001 0.001 0.001"/>
             </geometry>
             <material name="dark"/>
@@ -84,5 +84,5 @@
             <origin xyz="0 0 0" rpy="1.57 0 0"/>
             <geometry>
-                <mesh filename="file://$(find af_obstacle_avoidance_cpp)/model/meshes/wheels/right_tire.stl" scale="0.001 0.001 0.001"/>
+                <mesh filename="file://$(find af_obstacle_avoidance_py)/model/meshes/wheels/right_tire.stl" scale="0.001 0.001 0.001"/>
             </geometry>
             <material name="dark"/>
